File: KICAD_onboarding_devboard.kicad_sch (KiCad schematic)
At the start: 19 parts

Commit message: rev 2
Parts:
- removed J?: Conn_01x03_Socket, symbol Connector:Conn_01x03_Socket
- removed SW?: SW_SPST, symbol Switch:SW_SPST
- removed U?: TLV76133DCY, Package_TO_SOT_SMD:SOT-223-3_TabPin2, symbol Regulator_Linear:TLV76133DCY
- added C?: 10uF, symbol Device:C
- added C?: 470pF, symbol Device:C
- added C?: 6.8uF, symbol Device:C
- added C?: 2.2uF, symbol Device:C
- added C?: 1uF, symbol Device:C
- added J?: Conn_ST_STDC14, symbol Connector:Conn_ST_STDC14
- added J?: Conn_01x18_Pin, symbol Connector:Conn_01x18_Pin
- added PS?: ROE-1205S, ROE-1205S:CONV_ROE-1205S, symbol ROE-1205S:ROE-1205S
- added PS?: ROE-0505S, ROE-1205S:CONV_ROE-1205S, symbol ROE-1205S:ROE-1205S
- added R? (x4): 20k, symbol Device:R
- added R? (x4): 10k, symbol Device:R
- added R?: 4.7k, symbol Device:R
- added SW?: SW_Push_DPDT, symbol Switch:SW_Push_DPDT
- added SW?: SW_Push_Open, symbol Switch:SW_Push_Open
- added SW?: SW_Push, symbol Switch:SW_Push
- added U?: TLV76133DCYR, Package_TO_SOT_SMD:SOT-223-3_TabPin2, symbol Regulator_Linear:TLV76150DCY
Connections:
- net FDCAN_RX is gone; now on net FDCAN1_RX: U?.2 (RXD)
- net FDCAN_TX is gone; now on net FDCAN1_TX: U?.3 (TXD)
- net 3.3V: now also C?.1, J?.13 (Pin_13), SW?.2, SW?.2 (B), U?.2 (VO)
- net 5V: now also C?.1, C?.2, J?.14 (Pin_14), PS?.4 (+VOUT), PS?.4 (+VOUT), U?.3 (VI)
- net GND: now also C?.1, C?.1, C?.1, C?.1, C?.2, J?.12 (Pin_12), J?.5 (GND), J?.7 (GND), PS?.1 (-VIN), PS?.1 (-VIN), R?.2, R?.2, R?.2, R?.2, R?.2, U?.1 (GND); no longer C?.2
- net NRST: now also R?.1, SW?.1 (A)
- net SWCLK/BOOT0: now also J?.6 (JCLK/SWCLK), SW?.1
- net SWDIO: now also J?.4 (JTMS/SWDIO)
- net PA4/ADC_IN4: now reaches U?.15 (PA4)
- net PA4/ADC_IN4: now also R?.1, R?.2
- net PA5/ADC_IN5: now reaches U?.16 (PA5)
- net PA5/ADC_IN5: now also R?.1, R?.2
- net PA6/ADC_IN6: now reaches U?.17 (PA6)
- net PA6/ADC_IN6: now also R?.1, R?.2
- net PA7/ADC_IN7: now reaches U?.18 (PA7)
- net PA7/ADC_IN7: now also R?.1, R?.2
- net PB0/ADC_IN8: now reaches U?.19 (PB0)
- net PB0/ADC_IN8: now also J?.9 (Pin_9)
- net PB1/ADC_IN9: now reaches U?.20 (PB1)
- net PB1/ADC_IN9: now also J?.8 (Pin_8)
- net PB2/ADC_IN10: now reaches U?.21 (PB2)
- net PB2/ADC_IN10: now also J?.7 (Pin_7)
- net 3.3V_DIRTY: no longer names the net of U?.17 (3V3OUT), U?.4 (VCCIO)
- net 3.3V_DIRTY: now also C?.2; no longer C?.1
- net 5V_DIRTY renamed USB_5V_IN
- net USB_5V_IN: now also SW?.5 (B)
- net I2C1_SCL renamed PB6/I2C1_SCL
- net PB6/I2C1_SCL: now also J?.6 (Pin_6)
- net I2C1_SDA renamed PB7/I2C1_SDA
- net PB7/I2C1_SDA: now also J?.5 (Pin_5)
- net SPI2_MISO renamed PB14/SPI2_MISO
- net PB14/SPI2_MISO: now also J?.2 (Pin_2)
- net SPI2_MOSI renamed PB15/SPI2_MOSI
- net PB15/SPI2_MOSI: now also J?.1 (Pin_1)
- net SPI2_NSS renamed PB12/SPI2_NSS
- net PB12/SPI2_NSS: now also J?.4 (Pin_4)
- net SPI2_SCK renamed PB13/SPI2_SCK
- net PB13/SPI2_SCK: now also J?.3 (Pin_3)
- net USART4_RX renamed PA1/USART4_RX
- net USART4_TX renamed PA0/USART4_TX
- net PA0/USART4_TX: now also J?.11 (Pin_11)
- new net: J?.15 (Pin_15), R?.1
- new net: C?.2, C?.2, PS?.2 (+VIN), SW?.3 (C)
- new net: C?.2, PS?.2 (+VIN), SW?.4 (A)
- new net: J?.18 (Pin_18), R?.1
- new net: J?.17 (Pin_17), R?.1
- new net: J?.16 (Pin_16), R?.1
- new net 12V_IN: SW?.2 (B)
- new net PA1/USART4_TX: J?.10 (Pin_10)
- no-connect marks 17 -> 21
Other:
- note added: "*5v_dirty*"
- note added: "*please disconnect power when switching power modes lmao*"
- note added: "BOOT0->VCC: system memory (UART flash) BOOT0->GND: main flash memory *is this the right value for a pull-down?*"
- note added: "POWER"
- note added: "notes for aadi: STLINK - Should I be using more pins on the STDC header? from what I read this seems like all I need... POWER - Can I feed the outputs of both ROE chips into the 5V net like that? only one is gonna be switched on at a time so it seems fine to me... unsure if it could be a problem IO - Now that I think about it probably need to have 12V tolerant dedicated ADC headers - Will break o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"
- note removed: "*I don't think this connector is right...*"
- note removed: "BOOT0->VCC: system memory (UART flash) BOOT0->GND: main flash memory *is this the right value for a pull-down?* *should it be a pull-up?*"
- moved on the sheet: C?, R?
